Commit message: Mudanças finais. Funcionou!

File: src/robot_description/urdf/differential_robot.xacro (robot description, xacro)
@@ -1,8 +1,8 @@
 <?xml version="1.0"?>
 <robot xmlns:xacro="http://www.ros.org/wiki/xacro" name="dif_rob">
-    <xacro:property name="radius" value="0.3" />
-    <xacro:property name="height" value="0.08" />
-    <xacro:property name="mass" value="10.0" />
-    <xacro:property name="wheel_radius" value="0.08" />
+    <xacro:property name="radius" value="0.15" />
+    <xacro:property name="height" value="0.06" />
+    <xacro:property name="mass" value="6.0" />
+    <xacro:property name="wheel_radius" value="0.06" />
     <xacro:property name="casterBall_radius" value="${height/2-wheel_radius/4}" />
     <xacro:property name="lidarSup_height" value="${height/2-wheel_radius/4+0.05}"/>

File: src/robot_description/urdf/wheels.xacro (robot description, xacro)
@@ -2,5 +2,5 @@
 <robot xmlns:xacro="http://www.ros.org/wiki/xacro">
     <xacro:macro  name="wheel" params="prefix reflect base_width wheel_radius *axis">
-        <xacro:property name="wheel_len" value="0.1" />
+        <xacro:property name="wheel_len" value="0.05" />
         <xacro:property name="wheel_mass" value="0.5" />
         <link name="${prefix}_wheel">
